File: HARDWARE/Computadora/.kicad_pcb.kicad_pcb (KiCad board)
At the start: 2 copper layers, 82 x 87 mm, 45 parts, among them IC1 ATMEGA328-P, J1 DB9, K1 AUX_PINS, P1 MOTORS PWM OUTPUT, P2 CONN_2, P3 CONN_SENSORES, Q1 BS170, Q2 BS170, SW1 RESET, U1 MAX232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

Commit message: Se termina primera version del pcb. yeah!
Signed-off-by: Gonzalo Nahuel Vaca <vacagonzalo@gmail.com>
Parts:
- ICSP1: footprint pin_array_3x2corregido -> pin_array_3x2
- J1: footprint DB9FCcorregido -> DB9FC
- P1: footprint pin_array_6x2corregido -> pin_array_6x2
- moved D1 92.6 mm to (56.0, 85.0), turned to 270 degrees
- moved D2 92.5 mm to (56.0, 78.5), turned to 270 degrees
- moved RV1 85.9 mm to (84.5, 61.0)
- moved P3 85.0 mm to (95.0, 117.5)
- moved R10 82.2 mm to (93.0, 79.5)
- moved R5 82.2 mm to (93.0, 74.5)
- moved R6 82.2 mm to (93.0, 77.0)
- moved R8 82.2 mm to (93.0, 84.5)
- moved R9 82.2 mm to (93.0, 82.0)
- moved D5 81.8 mm to (102.0, 88.5), turned to 270 degrees
- moved IC1 81.8 mm to (79.0, 91.0)
- moved P1 81.5 mm to (79.0, 117.5), turned to 180 degrees
- moved R1 75.7 mm to (65.0, 79.5), turned to 180 degrees
- moved R2 75.7 mm to (65.0, 77.0), turned to 180 degrees
- moved JP1 75.3 mm to (65.5, 86.0), turned to 180 degrees
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Connections:
- ICSP1 pad 1: /SCK -> /MISO
- ICSP1 pad 2: /MISO -> +5V
- ICSP1 pad 3: +5V -> /SCK
- ICSP1 pad 5: GND -> /RESET
- ICSP1 pad 6: /RESET -> GND
- J1 pad : GND -> (no net)
- J1 pad 1: GND -> (no net)
- J1 pad 2: N-0000045 -> N-0000046
- J1 pad 3: N-0000046 -> N-0000045
- J1 pad 4: GND -> (no net)
- J1 pad 6: GND -> (no net)
- J1 pad 7: GND -> (no net)
- J1 pad 8: GND -> (no net)
- J1 pad 9: GND -> (no net)
- P1 pad 1: +5V -> GND
- P1 pad 10: /PWM1 -> GND
- P1 pad 11: GND -> +5V
- P1 pad 12: GND -> /PWM4
- P1 pad 2: /PWM3 -> +5V
- P1 pad 3: +5V -> /PWM1
- P1 pad 4: +5V -> GND
- P1 pad 6: /PWM4 -> /PWM2
- P1 pad 8: /PWM2 -> +5V
- P1 pad 9: GND -> /PWM3
Routing:
- net GND: track 489.5 -> 0.00 mm
- net +5V: track 371.5 -> 0.00 mm, vias 8 -> 0
- net +2.5V: track 115.7 -> 0.00 mm, vias 4 -> 0
- net /RESET: track 45.4 -> 0.00 mm
- net /SP: track 45.3 -> 0.00 mm
- net /MOSI: track 39.0 -> 0.00 mm
- net N-0000045: track 35.0 -> 0.00 mm
- net /SCK: track 34.7 -> 0.00 mm
- net /MISO: track 34.2 -> 0.00 mm
- net N-0000046: track 33.8 -> 0.00 mm
- net /PWM4: track 33.7 -> 0.00 mm
- net /RX: track 28.1 -> 0.00 mm, vias 2 -> 0
- net /TX: track 27.9 -> 0.00 mm, vias 2 -> 0
- net /XTAL2: track 24.7 -> 0.00 mm
- net /XTAL1: track 23.6 -> 0.00 mm
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Other:
- board outline removed
- net class Default: clearance 0.508 -> 0.254; trace_width 0.508 -> 0.254
- rule pad_to_mask_clearance: 0 -> 0.2
- rule trace_clearance: 0.508 -> 0.254
